Commit message: Update Zainetto_2.96_MOD10_DEF.urdf

File: zainetto/robot/Zainetto_2.96_MOD10_DEF.urdf (robot description, URDF)
Before this commit: robot zainetto, 1 links, 0 joints
Links:
- link base_link: geometry collision mesh filename=package://zainetto/meshes/Zainetto_2.96_MOD10_DEF.stl scale=0.001 0.001 0.001; visual mesh filename=package://zainetto/meshes/Zainetto_2.96_MOD10_DEF.stl scale=0.001 0.001 0.001
