Commit message: Update Zainetto_2_96_MOD10_DEF.urdf

File: zainetto/robot/Zainetto_2_96_MOD10_DEF.urdf (robot description, URDF)
Before this commit: robot zainetto, 1 links, 0 joints
Links:
- link base_link: geometry collision mesh filename=package://your_package_name/meshes/Zainetto_2_96_MOD10_DEF.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 scale=0.001 0.001 0.001; visual mesh filename=package://your_package_name/meshes/Zainetto_2_96_MOD10_DEF.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 scale=0.001 0.001 0.001
